File: Alice Plate/Alice Plate.kicad_pcb (KiCad board)
At the start: 2 copper layers, 338.8 x 123.9 mm, 65 parts

Commit message: make plate changes
Parts:
- removed the REF** at (-1.10, 109.7)
Changed lines of the file:
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@@
     (tracks 0)
     (zones 0)
-    (modules 65)
+    (modules 64)
     (nets 1)
   )
@@
     (fp_arc (start 6.5 6.5) (end 6.499999 7) (angle -90) (layer Edge.Cuts) (width 0.15))
   )
-  (module Graphics:audrentis_copper (layer F.Cu)
-    (at -1.102208 109.716114)
-    (fp_text reference REF** (at 0 0.5) (layer B.Fab)
-      (effects (font (size 1 1) (thickness 0.15)) (justify mirror))
-    )
-    (fp_text value audrentis_copper (at 0 -0.5) (layer F.Fab)
-      (effects (font (size 1 1) (thickness 0.15)))
-    )
-    (fp_line (start -6.25 2) (end 6.75 2) (layer F.Mask) (width 0.6))
-    (fp_line (start -6.25 1.5) (end 6.75 1.5) (layer F.Mask) (width 0.6))
-    (fp_line (start -6.25 1) (end 6.75 1) (layer F.Mask) (width 0.6))
-    (fp_line (start -6.25 0.5) (end 6.75 0.5) (layer F.Mask) (width 0.6))
-    (fp_line (start -6.25 0.25) (end 6.75 0.25) (layer F.Mask) (width 0.6))
-    (fp_line (start -6.25 -0.25) (end 6.75 -0.25) (layer F.Mask) (width 0.6))
-    (fp_line (start -6.25 -0.75) (end 6.75 -0.75) (layer F.Mask) (width 0.6))
-    (fp_line (start -6.25 -1) (end 6.75 -1) (layer F.Mask) (width 0.6))
-    (fp_line (start -6.25 -1.5) (end 6.75 -1.5) (layer F.Mask) (width 0.6))
-    (fp_line (start -6.25 -2) (end 6.75 -2) (layer F.Mask) (width 0.6))
-    (fp_line (start -6.5 2.25) (end 6.5 2.25) (layer F.Mask) (width 0.6))
-    (fp_line (start -6.75 2) (end 6.25 2) (layer F.Mask) (width 0.6))
-    (fp_line (start -6.75 1.5) (end 6.25 1.5) (layer F.Mask) (width 0.6))
-    (fp_line (start -6.75 1) (end 6.25 1) (layer F.Mask) (width 0.6))
-    (fp_line (start -6.75 0.5) (end 6.25 0.5) (layer F.Mask) (width 0.6))
-    (fp_line (start -6.75 0) (end 6.25 0) (layer F.Mask) (width 0.6))
-    (fp_line (start -6.75 -0.5) (end 6.25 -0.5) (layer F.Mask) (width 0.6))
-    (fp_line (start -6.75 -1) (end 6.25 -1) (layer F.Mask) (width 0.6))
-    (fp_line (start -6.75 -1.5) (end 6.25 -1.5) (layer F.Mask) (width 0.6))
-    (fp_line (start -6.75 -2) (end 6.25 -2) (layer F.Mask) (width 0.6))
-    (fp_line (start -6.5 -2.25) (end 6.5 -2.25) (layer F.Mask) (width 0.6))
-    (fp_text user audrentis.xyz (at 0 0) (layer F.Cu)
-      (effects (font (size 1.35 1.35) (thickness 0.29)))
-    )
-    (fp_text user audrentis.xyz (at 0 0) (layer F.Mask)
-      (effects (font (size 1.35 1.35) (thickness 0.29)))
-    )
-    (fp_arc (start -6.25 -1.75) (end -6.25 -2.5) (angle -90) (layer F.Mask) (width 0.25))
-    (fp_line (start -7 -1.75) (end -7 1.75) (layer F.Mask) (width 0.25))
-    (fp_arc (start -6.25 1.75) (end -7 1.75) (angle -90) (layer F.Mask) (width 0.25))
-    (fp_line (start -6.25 2.5) (end 6.25 2.5) (layer F.Mask) (width 0.25))
-    (fp_arc (start 6.25 1.75) (end 6.25 2.5) (angle -90) (layer F.Mask) (width 0.25))
-    (fp_line (start 7 -1.75) (end 7 1.75) (layer F.Mask) (width 0.25))
-    (fp_arc (start 6.25 -1.75) (end 7 -1.75) (angle -90) (layer F.Mask) (width 0.25))
-    (fp_line (start 6.25 -2.5) (end -6.25 -2.5) (layer F.Mask) (width 0.25))
-    (fp_line (start 6.25 -2.5) (end -6.25 -2.5) (layer F.Cu) (width 0.25))
-    (fp_line (start 7 -1.75) (end 7 1.75) (layer F.Cu) (width 0.25))
-    (fp_line (start -6.25 2.5) (end 6.25 2.5) (layer F.Cu) (width 0.25))
-    (fp_line (start -7 -1.75) (end -7 1.75) (layer F.Cu) (width 0.25))
-    (fp_arc (start 6.25 1.75) (end 6.25 2.5) (angle -90) (layer F.Cu) (width 0.25))
-    (fp_arc (start 6.25 -1.75) (end 7 -1.75) (angle -90) (layer F.Cu) (width 0.25))
-    (fp_arc (start -6.25 1.75) (end -7 1.75) (angle -90) (layer F.Cu) (width 0.25))
-    (fp_arc (start -6.25 -1.75) (end -6.25 -2.5) (angle -90) (layer F.Cu) (width 0.25))
-  )
   (module MX_Plate_Cutouts:1.5u (layer F.Cu)
